Commit message: add X2 EDU robot models, update stl and urdf params

File: X2_URDF-v1.3.0/x2_fist.urdf (robot description, URDF)
Before this commit: robot x2_fist, 35 links, 34 joints
Joints:
- joint head_yaw_joint: limit lower=-0.366 upper=0.366 effort=2.6 velocity=6.019 -> lower=-0.349 upper=0.349 effort=2.6 velocity=6.019
- joint left_ankle_roll_joint: limit lower=-0.262 upper=0.262 effort=24 velocity=15.077 -> lower=-0.2967 upper=0.2967 effort=24 velocity=15.077
- joint left_hip_yaw_joint: limit lower=-1.684 upper=3.43 effort=120 velocity=11.936 -> lower=-1.8588 upper=3.6041 effort=120 velocity=11.936
- joint left_shoulder_roll_joint: limit lower=-0.061 upper=2.993 effort=36 velocity=13.088 -> lower=-0.061 upper=3.0456 effort=36 velocity=13.088
- joint right_ankle_roll_joint: limit lower=-0.2625 upper=0.2625 effort=24 velocity=15.077 -> lower=-0.2967 upper=0.2967 effort=24 velocity=15.077
- joint right_hip_yaw_joint: limit lower=-3.43 upper=1.684 effort=120 velocity=11.936 -> lower=-3.6041 upper=1.8588 effort=120 velocity=11.936
- joint right_shoulder_roll_joint: limit lower=-2.993 upper=0.061 effort=36 velocity=13.088 -> lower=-3.0456 upper=0.061 effort=36 velocity=13.088
- joint waist_yaw_joint: limit lower=-3.43 upper=2.382 effort=120 velocity=11.936 -> lower=-3.43 upper=2.2078 effort=120 velocity=11.936

File: X2_URDF-v1.3.0/x2_ultra.urdf (robot description, URDF)
Before this commit: robot x2_ultra, 41 links, 40 joints
Joints:
- joint head_yaw_joint: limit lower=-0.366 upper=0.366 effort=2.6 velocity=6.019 -> lower=-0.349 upper=0.349 effort=2.6 velocity=6.019
- joint left_ankle_roll_joint: limit lower=-0.262 upper=0.262 effort=24 velocity=15.077 -> lower=-0.2967 upper=0.2967 effort=24 velocity=15.077
- joint left_hip_yaw_joint: limit lower=-1.684 upper=3.43 effort=120 velocity=11.936 -> lower=-1.8588 upper=3.6041 effort=120 velocity=11.936
- joint left_shoulder_roll_joint: limit lower=-0.061 upper=2.993 effort=36 velocity=13.088 -> lower=-0.061 upper=3.0456 effort=36 velocity=13.088
- joint left_wrist_pitch_joint: limit lower=-0.558 upper=0.558 effort=4.8 velocity=4.188 -> lower=-0.5236 upper=0.5236 effort=4.8 velocity=4.188
- joint left_wrist_roll_joint: limit lower=-1.571 upper=0.724 effort=4.8 velocity=4.188 -> lower=-1.5097 upper=0.724 effort=4.8 velocity=4.188
- joint right_ankle_roll_joint: limit lower=-0.2625 upper=0.2625 effort=24 velocity=15.077 -> lower=-0.2967 upper=0.2967 effort=24 velocity=15.077
- joint right_hip_yaw_joint: limit lower=-3.43 upper=1.684 effort=120 velocity=11.936 -> lower=-3.6041 upper=1.8588 effort=120 velocity=11.936
- joint right_shoulder_roll_joint: limit lower=-2.993 upper=0.061 effort=36 velocity=13.088 -> lower=-3.0456 upper=0.061 effort=36 velocity=13.088
- joint right_wrist_pitch_joint: limit lower=-0.558 upper=0.558 effort=4.8 velocity=4.188 -> lower=-0.5236 upper=0.5236 effort=4.8 velocity=4.188
- joint right_wrist_roll_joint: limit lower=-0.724 upper=1.571 effort=4.8 velocity=4.188 -> lower=-0.724 upper=1.5097 effort=4.8 velocity=4.188
- joint waist_yaw_joint: limit lower=-3.43 upper=2.382 effort=120 velocity=11.936 -> lower=-3.43 upper=2.2078 effort=120 velocity=11.936

File: X2_URDF-v1.3.0/x2_ultra_simple_collision.urdf (robot description, URDF)
Before this commit: robot x2_ultra_simple_collision, 39 links, 38 joints
Links:
- link rgb_head_center: geometry visual mesh filename=./meshes/rgb_head_center_link.STL
- link rgb_head_rear: geometry visual mesh filename=./meshes/rgb_head_rear_link.STL
- link rgbd_head_front: geometry visual mesh filename=./meshes/rgbd_head_front_link.STL
- link stereo_head_front: geometry visual mesh filename=./meshes/stereo_head_front_link.STL
Joints:
- joint head_yaw_joint: limit lower=-0.366 upper=0.366 effort=2.6 velocity=6.019 -> lower=-0.349 upper=0.349 effort=2.6 velocity=6.019
- joint left_ankle_roll_joint: limit lower=-0.262 upper=0.262 effort=24 velocity=15.077 -> lower=-0.2967 upper=0.2967 effort=24 velocity=15.077
- joint left_hip_yaw_joint: limit lower=-1.684 upper=3.43 effort=120 velocity=11.936 -> lower=-1.8588 upper=3.6041 effort=120 velocity=11.936
- joint left_shoulder_roll_joint: limit lower=-0.061 upper=2.993 effort=36 velocity=13.088 -> lower=-0.061 upper=3.0456 effort=36 velocity=13.088
- joint left_wrist_pitch_joint: limit lower=-0.558 upper=0.558 effort=4.8 velocity=4.188 -> lower=-0.5236 upper=0.5236 effort=4.8 velocity=4.188
- joint left_wrist_roll_joint: limit lower=-1.571 upper=0.724 effort=4.8 velocity=4.188 -> lower=-1.5097 upper=0.724 effort=4.8 velocity=4.188
- joint right_ankle_roll_joint: limit lower=-0.2625 upper=0.2625 effort=24 velocity=15.077 -> lower=-0.2967 upper=0.2967 effort=24 velocity=15.077
- joint right_hip_yaw_joint: limit lower=-3.43 upper=1.684 effort=120 velocity=11.936 -> lower=-3.6041 upper=1.8588 effort=120 velocity=11.936
- joint right_shoulder_roll_joint: limit lower=-2.993 upper=0.061 effort=36 velocity=13.088 -> lower=-3.0456 upper=0.061 effort=36 velocity=13.088
- joint right_wrist_pitch_joint: limit lower=-0.558 upper=0.558 effort=4.8 velocity=4.188 -> lower=-0.5236 upper=0.5236 effort=4.8 velocity=4.188
- joint right_wrist_roll_joint: limit lower=-0.724 upper=1.571 effort=4.8 velocity=4.188 -> lower=-0.724 upper=1.5097 effort=4.8 velocity=4.188
- joint waist_yaw_joint: limit lower=-3.43 upper=2.382 effort=120 velocity=11.936 -> lower=-3.43 upper=2.2078 effort=120 velocity=11.936

File: X2_URDF-v1.4.0/X2-EDU.urdf (robot description, URDF)
Before this commit: robot X2-Ultra, 39 links, 38 joints
Links:
- removed link head_pitch_link
- removed link head_yaw_link
- removed link lidar_chest_front_link
- removed link rgb_head_center_link
- removed link rgb_head_rear_link
- removed link rgbd_head_front_link
- removed link stereo_head_front_link
- link left_ankle_pitch_link: mass 0.949 -> 0.94912290; geometry collision mesh filename=./meshes/left_ankle_pitch_link.stl; visual mesh filename=./meshes/left_ankle_pitch_link.stl
- link left_ankle_roll_link: mass 1.048 -> 1.04791701; geometry collision mesh filename=./meshes/left_ankle_roll_link.stl; visual mesh filename=./meshes/left_ankle_roll_link.stl
- link left_elbow_link: mass 0.675 -> 0.62333677
- link left_hip_pitch_link: mass 1.474 -> 1.47374636; geometry collision mesh filename=./meshes/left_hip_pitch_link.stl; visual mesh filename=./meshes/left_hip_pitch_link.stl
- link left_hip_roll_link: mass 1.667 -> 1.52722346; geometry collision mesh filename=./meshes/left_hip_roll_link.stl; visual mesh filename=./meshes/left_hip_roll_link.stl
- link left_hip_yaw_link: mass 2.087 -> 1.88769448; geometry collision mesh filename=./meshes/left_hip_yaw_link.stl; visual mesh filename=./meshes/left_hip_yaw_link.stl
- link left_knee_link: mass 1.838 -> 1.66317142
- link left_shoulder_pitch_link: mass 0.927 -> 0.92680928; geometry collision mesh filename=./meshes/left_shoulder_pitch_link.stl; visual mesh filename=./meshes/left_shoulder_pitch_link.stl
- link left_shoulder_roll_link: mass 0.741 -> 0.68561752; geometry collision mesh filename=./meshes/left_shoulder_roll_link.stl; visual mesh filename=./meshes/left_shoulder_roll_link.stl
- link left_shoulder_yaw_link: mass 0.703 -> 0.64753096; geometry collision mesh filename=./meshes/left_shoulder_yaw_link.stl; visual mesh filename=./meshes/left_shoulder_yaw_link.stl
- link left_wrist_pitch_link: mass 0.344 -> 0.34431419; geometry collision mesh filename=./meshes/left_wrist_pitch_link.stl; visual mesh filename=./meshes/left_wrist_pitch_link.stl
- link left_wrist_roll_link: mass 0.338 -> 0.33766760
- link left_wrist_yaw_link: mass 0.37 -> 0.32664866; geometry collision mesh filename=./meshes/left_wrist_yaw_link.stl; visual mesh filename=./meshes/left_wrist_yaw_link.stl
- link pelvis: mass 3.59 -> 3.59010086; geometry collision mesh filename=./meshes/pelvis.stl; visual mesh filename=./meshes/pelvis.stl
- link right_ankle_pitch_link: mass 0.948 -> 0.94783305; geometry collision mesh filename=./meshes/right_ankle_pitch_link.stl; visual mesh filename=./meshes/right_ankle_pitch_link.stl
- link right_ankle_roll_link: mass 1.046 -> 1.04608350; geometry collision mesh filename=./meshes/right_ankle_roll_link.stl; visual mesh filename=./meshes/right_ankle_roll_link.stl
- link right_elbow_link: mass 0.674 -> 0.62244416
- link right_hip_pitch_link: mass 1.476 -> 1.47631288; geometry collision mesh filename=./meshes/right_hip_pitch_link.stl; visual mesh filename=./meshes/right_hip_pitch_link.stl
- link right_hip_roll_link: mass 1.669 -> 1.52896200; geometry collision mesh filename=./meshes/right_hip_roll_link.stl; visual mesh filename=./meshes/right_hip_roll_link.stl
- link right_hip_yaw_link: mass 2.072 -> 1.87281245; geometry collision mesh filename=./meshes/right_hip_yaw_link.stl; visual mesh filename=./meshes/right_hip_yaw_link.stl
- link right_knee_link: mass 1.826 -> 1.65057226
- link right_shoulder_pitch_link: mass 0.936 -> 0.93606401; geometry collision mesh filename=./meshes/right_shoulder_pitch_link.stl; visual mesh filename=./meshes/right_shoulder_pitch_link.stl
- link right_shoulder_roll_link: mass 0.73 -> 0.67523132; geometry collision mesh filename=./meshes/right_shoulder_roll_link.stl; visual mesh filename=./meshes/right_shoulder_roll_link.stl
- link right_shoulder_yaw_link: mass 0.696 -> 0.64129141; geometry collision mesh filename=./meshes/right_shoulder_yaw_link.stl; visual mesh filename=./meshes/right_shoulder_yaw_link.stl
- link right_wrist_pitch_link: mass 0.336 -> 0.33614452; geometry collision mesh filename=./meshes/right_wrist_pitch_link.stl; visual mesh filename=./meshes/right_wrist_pitch_link.stl
- link right_wrist_roll_link: mass 0.337 -> 0.33733146
- link right_wrist_yaw_link: mass 0.373 -> 0.33028980; geometry collision mesh filename=./meshes/right_wrist_yaw_link.stl; visual mesh filename=./meshes/right_wrist_yaw_link.stl
- link torso_link: mass 10.986 -> 10.59420745; geometry collision mesh filename=./meshes/torso_lite_link.stl; visual mesh filename=./meshes/torso_lite_link.stl
- link waist_pitch_link: mass 0.42 -> 0.42036568; geometry collision mesh filename=./meshes/waist_pitch_link.stl; visual mesh filename=./meshes/waist_pitch_link.stl
- link waist_yaw_link: mass 1.788 -> 1.75326322; geometry collision mesh filename=./meshes/waist_yaw_link.stl; visual mesh filename=./meshes/waist_yaw_link.stl
Joints:
- removed joint head_pitch_joint
- removed joint head_yaw_joint
- removed joint lidar_chest_front_joint
- removed joint rgb_head_center_joint
- removed joint rgb_head_rear_joint
- removed joint rgbd_head_front_joint
- removed joint stereo_head_front_joint
- joint imu_in_pelvis_joint: origin xyz=0.024072 -0.0019436 0.04011 rpy=-3.1416 0 0 -> xyz=0.0240720441523812 -0.00194358848977061 0.0401099955799955 rpy=-3.14159265358979 0 0
- joint left_hip_pitch_joint: origin xyz=0 0.07135 0 rpy=0 0 0 -> xyz=0 0.0713499999999883 0 rpy=0 0 0
- joint left_hip_roll_joint: origin xyz=-0.00057492 0.0657 0 rpy=0 0 0 -> xyz=-0.000574923873940869 0.0656999999999472 0 rpy=0 0 0
- joint right_shoulder_pitch_joint: origin xyz=0.0032597 -0.14292 0.24172 rpy=-0.20945 0 0 -> xyz=0.00325970359616329 -0.142916758596713 0.241717525178737 rpy=-0.209449427348634 0 0

File: X2_URDF-v1.4.0/X2-EDU_simple_collision.urdf (robot description, URDF)
Before this commit: robot X2-Ultra, 39 links, 38 joints
Links:
- removed link head_pitch_link
- removed link head_yaw_link
- removed link lidar_chest_front_link
- removed link rgb_head_center_link
- removed link rgb_head_rear_link
- removed link rgbd_head_front_link
- removed link stereo_head_front_link
- link left_ankle_pitch_link: mass 0.949 -> 0.94912290
- link left_ankle_roll_link: mass 1.048 -> 1.04791701
- link left_elbow_link: mass 0.675 -> 0.62333677
- link left_hip_pitch_link: mass 1.474 -> 1.47374636
- link left_hip_roll_link: mass 1.667 -> 1.52722346
- link left_hip_yaw_link: mass 2.087 -> 1.88769448
- link left_knee_link: mass 1.838 -> 1.66317142
- link left_shoulder_pitch_link: mass 0.927 -> 0.92680928
- link left_shoulder_roll_link: mass 0.741 -> 0.68561752
- link left_shoulder_yaw_link: mass 0.703 -> 0.64753096
- link left_wrist_pitch_link: mass 0.344 -> 0.34431419
- link left_wrist_roll_link: mass 0.338 -> 0.33766760
- link left_wrist_yaw_link: mass 0.37 -> 0.32664866
- link pelvis: mass 3.59 -> 3.59010086
- link right_ankle_pitch_link: mass 0.948 -> 0.94783305
- link right_ankle_roll_link: mass 1.046 -> 1.04608350
- link right_elbow_link: mass 0.674 -> 0.62244416
- link right_hip_pitch_link: mass 1.476 -> 1.47631288
- link right_hip_roll_link: mass 1.669 -> 1.52896200
- link right_hip_yaw_link: mass 2.072 -> 1.87281245
- link right_knee_link: mass 1.826 -> 1.65057226
- link right_shoulder_pitch_link: mass 0.936 -> 0.93606401
- link right_shoulder_roll_link: mass 0.73 -> 0.67523132
- link right_shoulder_yaw_link: mass 0.696 -> 0.64129141
- link right_wrist_pitch_link: mass 0.336 -> 0.33614452
- link right_wrist_roll_link: mass 0.337 -> 0.33733146
- link right_wrist_yaw_link: mass 0.373 -> 0.33028980
- link torso_link: mass 10.986 -> 10.59420745; geometry collision cylinder length=0.08 radius=0.08; collision mesh filename=./meshes/torso_lite_link.stl
- link waist_pitch_link: mass 0.42 -> 0.42036568
- link waist_yaw_link: mass 1.788 -> 1.75326322
Joints:
- removed joint head_pitch_joint
- removed joint head_yaw_joint
- removed joint lidar_chest_front_joint
- removed joint rgb_head_center_joint
- removed joint rgb_head_rear_joint
- removed joint rgbd_head_front_joint
- removed joint stereo_head_front_joint
- joint imu_in_pelvis_joint: origin xyz=0.024072 -0.0019436 0.04011 rpy=-3.1416 0 0 -> xyz=0.0240720441523812 -0.00194358848977061 0.0401099955799955 rpy=-3.14159265358979 0 0
- joint left_hip_pitch_joint: origin xyz=0 0.07135 0 rpy=0 0 0 -> xyz=0 0.0713499999999883 0 rpy=0 0 0
- joint left_hip_roll_joint: origin xyz=-0.00057492 0.0657 0 rpy=0 0 0 -> xyz=-0.000574923873940869 0.0656999999999472 0 rpy=0 0 0
- joint right_shoulder_pitch_joint: origin xyz=0.0032597 -0.14292 0.24172 rpy=-0.20945 0 0 -> xyz=0.00325970359616329 -0.142916758596713 0.241717525178737 rpy=-0.209449427348634 0 0

File: X2_URDF-v1.4.0/X2-Ultra.urdf (robot description, URDF)
Before this commit: robot X2-Ultra, 39 links, 38 joints
Joints:
- joint head_pitch_joint: limit lower=-0.523599 upper=0.523599 effort=2.3 velocity=10.472 -> lower=-0.401425 upper=0.488692 effort=2 velocity=10.472
- joint head_yaw_joint: limit lower=-0.488692 upper=0.488692 effort=2.3 velocity=10.472 -> lower=-0.488692 upper=0.488692 effort=3.13125 velocity=3.3109
- joint left_ankle_roll_joint: limit lower=-0.261799 upper=0.261799 effort=36 velocity=14.660799999999998 -> lower=-0.2967059728 upper=0.2967059728 effort=36 velocity=14.660799999999998
- joint left_hip_yaw_joint: limit lower=-1.684243 upper=3.429572 effort=120 velocity=11.93808 -> lower=-1.858775925 upper=3.604104925 effort=120 velocity=11.93808
- joint left_shoulder_roll_joint: limit lower=-0.061087 upper=2.984513 effort=60 velocity=13.6136 -> lower=-0.061087 upper=3.045600 effort=60 velocity=13.6136
- joint right_ankle_roll_joint: limit lower=-0.261799 upper=0.261799 effort=36 velocity=14.660799999999998 -> lower=-0.2967059728 upper=0.2967059728 effort=36 velocity=14.660799999999998
- joint right_hip_yaw_joint: limit lower=-3.429572 upper=1.684243 effort=120 velocity=11.93808 -> lower=-3.604104925 upper=1.858775925 effort=120 velocity=11.93808
- joint right_shoulder_roll_joint: limit lower=-2.984513 upper=0.061087 effort=60 velocity=13.6136 -> lower=-3.045600 upper=0.061087 effort=60 velocity=13.6136
- joint waist_pitch_joint: limit lower=-0.488692 upper=0.488692 effort=36 velocity=14.660799999999998 -> lower=-0.314159 upper=0.314159 effort=36 velocity=14.660799999999998
- joint waist_roll_joint: limit lower=-0.488 upper=0.488 effort=36 velocity=13.088 -> lower=-0.488692 upper=0.488692 effort=36 velocity=14.661
- joint waist_yaw_joint: limit lower=-3.429572 upper=2.111848 effort=120 velocity=11.93808 -> lower=-3.429572 upper=2.120575 effort=120 velocity=11.93808
